Commit message: - packages needed.txt edited - bot with lidar added - slam and nav files required configured

File: bot/urdf/bot.xacro (robot description, xacro)
@@ -1,240 +1,87 @@
 <?xml version="1.0"?>
-<robot xmlns:xacro="http://www.ros.org/wiki/xacro"  name="diff_drive_bot" >
-<!-- Body dimensions-->
-<xacro:property name="length" value="0.6"/>
-<xacro:property name="bred" value="0.4"/>
-<xacro:property name="height" value="0.3"/>
-<!-- Wheel dims -->
-<xacro:property name="wheel_radius" value="0.05"/>
-<xacro:property name="wheel_length" value="0.1"/>
-<xacro:property name="wheel_z" value="-0.15"/>
-<!--Material density-->
-<xacro:property name="body_density" value="2710.0"/>
-<xacro:property name="wheel_density" value="2710.0"/>
-<!--Pi constant-->
-<xacro:property name="pi_const" value="3.14159265"/>
-<!--Robot body and wheel mass-->
-<xacro:property name="body_mass" value="${body_density*length*bred*height}"/>
-<xacro:property name="wheel_mass" value="${wheel_density*pi_const*wheel_radius*wheel_radius*wheel_length}"/>
-<!-- Moment of inertia of the wheel -->
-<xacro:property name="Iz_wheel" value="${0.5*wheel_mass*wheel_radius*wheel_length}"/>
-<xacro:property name="I_wheel" value="${(1.0/12.0)*wheel_mass*(3.0*wheel_radius*wheel_radius + wheel_length*wheel_length)}"/>
-<!-- macro defining inertial section of the wheel-->
-<xacro:macro name = "inertial_wheel">
-    <inertial>
-    <origin rpy = '0 0 0' xyz= '0 0 0'/>
-    <mass value = '${wheel_mass}'/>
-    <inertia ixx = "${I_wheel}" ixy="0.0" ixz = "0.0" iyy = "${I_wheel}" iyz="0" izz="${Iz_wheel}"/>
-    </inertial>
-</xacro:macro>
-<xacro:macro name="inertial_cylinder" params="mass length radius">
-  <inertial>
-    <mass value="${mass}"/>
-    <inertia ixx="${(1/12) * mass * (3*radius*radius + length*length)}" ixy="0.0" ixz="0.0"
-                    iyy="${(1/12) * mass * (3*radius*radius + length*length)}" iyz="0.0"
-                    izz="${(1/2) * mass * (radius*radius)}" />
-  </inertial>
-</xacro:macro>
-<!--control driver with gazebo-->
-<xacro:include filename="$(find bot)/urdf/bot.gazebo"/>
-<!--footprint link-->
-<link name="base_footprint"></link>
-<joint name="body_link_joint" type="fixed">
-  <parent link="base_footprint"/>
-  <child link="base_link"/>
-</joint>
-<!-- Body of the robot -->
-<link name="base_link">
-    <visual>
-        <geometry>
-          <box size="${length} ${bred} ${height}"/>
-        </geometry>
-        <material name="black">
-            <color rgba="0 0 0 1"/>
-        </material>
-    </visual>
-    <collision>
-        <geometry>
-            <box size="${length} ${bred} ${height}"/>
-        </geometry>
-        <origin rpy="0 0 0" xyz="0 0 0"/>
-    </collision>
-    <inertial>
-        <mass value = "${body_mass}"/>
-        <inertia
-            ixx = "${(1.0/12.0)*body_mass*(bred*bred + height*height)}" ixy = "0"
-            ixz = "0" iyy = "${(1.0/12.0)*body_mass*(length*length + height*height)}"
-            iyz ="0"
-            izz = "${(1.0/12.0)*body_mass*(bred*bred + length*length)}"/>
-    </inertial>
-</link>
-<!-- Joint Definition for right back wheel -->
-  <joint name="right_wheel_joint_back" type="continuous">
-    <parent link="base_link"/>
-    <child link="right_wheel_back"/>
-    <origin xyz="${-length/2+1.2*wheel_radius} ${-bred/2 - wheel_length/2} ${wheel_z}" rpy="0 0 0"/>
-    <axis xyz="0 1 0"/>
-    <limit effort="1000" velocity="1000"/>
-    <dynamics damping="1.0" friction="1.0"/>
-  </joint>
-  <!--  right back wheel -->
-  <link name="right_wheel_back">
-    <visual>
-    <origin rpy = '1.570795 0 0' xyz = '0 0 0'/>
-      <geometry>
-        <cylinder radius="${wheel_radius}" length="${wheel_length}"/> <!-- 100mm diameter wheel -->
-      </geometry>
-      <material name="grey">
-      <color rgba = '0.5 0.5 0.5 1'/>
-      </material>
-    </visual>
-    <collision>
-      <geometry>
-        <cylinder radius="${wheel_radius}" length="${wheel_length}"/>
-      </geometry>
-      <origin rpy = '1.570795 0 0' xyz = '0 0 0'/>
-    </collision>
-    <xacro:inertial_wheel/>
-  </link>
-<!-- Joint Definition for left back wheel -->
-  <joint name="left_wheel_joint_back" type="continuous">
-    <parent link="base_link"/>
-    <child link="left_wheel_back"/>
-    <origin xyz="${-length/2+1.2*wheel_radius} ${bred/2 + wheel_length/2} ${wheel_z}" rpy="0 0 0"/>
-    <axis xyz="0 1 0"/>
-    <limit effort="1000" velocity="1000"/>
-    <dynamics damping="1.0" friction="1.0"/>
-  </joint>
-  <!--  left back wheel -->
-  <link name="left_wheel_back">
-    <visual>
-    <origin rpy = '1.570795 0 0' xyz = '0 0 0'/>
-      <geometry>
-        <cylinder radius="${wheel_radius}" length="${wheel_length}"/> <!-- 100mm diameter wheel -->
-      </geometry>
-      <material name="grey">
-      <color rgba = '0.5 0.5 0.5 1'/>
-      </material>
-    </visual>
-    <collision>
-      <geometry>
-        <cylinder radius="${wheel_radius}" length="${wheel_length}"/>
-      </geometry>
-      <origin rpy = '1.570795 0 0' xyz = '0 0 0'/>
-    </collision>
-    <xacro:inertial_wheel/>
-  </link>
-<!-- Joint Definition for right front wheel -->
-  <joint name="right_wheel_joint_front" type="continuous">
-    <parent link="base_link"/>
-    <child link="right_wheel_front"/>
-    <origin xyz="${length/2-1.2*wheel_radius} ${-bred/2 - wheel_length/2} ${wheel_z}" rpy="0 0 0"/>
-    <axis xyz="0 1 0"/>
-    <limit effort="1000" velocity="1000"/>
-    <dynamics damping="1.0" friction="1.0"/>
-  </joint>
-  <!--  right front wheel -->
-  <link name="right_wheel_front">
-    <visual>
-    <origin rpy = '1.570795 0 0' xyz = '0 0 0'/>
-      <geometry>
-        <cylinder radius="${wheel_radius}" length="${wheel_length}"/> <!-- 100mm diameter wheel -->
-      </geometry>
-      <material name="grey">
-      <color rgba = '0.5 0.5 0.5 1'/>
-      </material>
-    </visual>
-    <collision>
-      <geometry>
-        <cylinder radius="${wheel_radius}" length="${wheel_length}"/>
-      </geometry>
-      <origin rpy = '1.570795 0 0' xyz = '0 0 0'/>
-    </collision>
-    <xacro:inertial_wheel/>
-  </link>
-  <!-- Joint Definition for left front wheel -->
-  <joint name="left_wheel_joint_front" type="continuous">
-    <parent link="base_link"/>
-    <child link="left_wheel_front"/>
-    <origin xyz="${length/2-1.2*wheel_radius} ${bred/2 + wheel_length/2} ${wheel_z}" rpy="0 0 0"/>
-    <axis xyz="0 1 0"/>
-    <limit effort="1000" velocity="1000"/>
-    <dynamics damping="1.0" friction="1.0"/>
-  </joint>
-  <!--  left front wheel -->
-  <link name="left_wheel_front">
-    <visual>
-    <origin rpy = '1.570795 0 0' xyz = '0 0 0'/>
-      <geometry>
-        <cylinder radius="${wheel_radius}" length="${wheel_length}"/> <!-- 100mm diameter wheel -->
-      </geometry>
-      <material name="grey">
-      <color rgba = '0.5 0.5 0.5 1'/>
-      </material>
-    </visual>
-    <collision>
-      <geometry>
-        <cylinder radius="${wheel_radius}" length="${wheel_length}"/>
-      </geometry>
-      <origin rpy = '1.570795 0 0' xyz = '0 0 0'/>
-    </collision>
-    <xacro:inertial_wheel/>
-  </link>
-  <!-- LiDAR Sensor -->
-<link name="lidar_link">
-  <visual>
-    <geometry>
-      <cylinder radius="0.05" length="0.1"/>
-    </geometry>
-    <material name="blue">
-      <color rgba="0 0 1 1"/>
-    </material>
-  </visual>
-  <collision>
-    <geometry>
-      <cylinder radius="0.05" length="0.1"/>
-    </geometry>
-  </collision>
-  <inertial>
-    <mass value="0.1"/>
-    <inertia ixx="0.001" ixy="0.0" ixz="0.0" iyy="0.001" iyz="0.0" izz="0.001"/>
-  </inertial>
-</link>
-<joint name="lidar_joint" type="fixed">
-  <parent link="base_link"/>
-  <child link="lidar_link"/>
-  <origin xyz="0.3 0 0.15" rpy="0 0 0"/>
-</joint>
-<!-- Gazebo LiDAR Plugin -->
-<gazebo reference="lidar_link">
-  <sensor type="ray" name="lidar_sensor">
-    <pose>0 0 0 0 0 0</pose>
-    <visualize>true</visualize>
-    <update_rate>10</update_rate>
-    <ray>
-      <scan>
-        <horizontal>
-          <samples>360</samples>
-          <resolution>1.0</resolution>
-          <min_angle>-3.14159</min_angle>
-          <max_angle>3.14159</max_angle>
-        </horizontal>
-      </scan>
-      <range>
-        <min>0.1</min>
-        <max>10.0</max>
-        <resolution>0.01</resolution>
-      </range>
-      <noise>
-        <type>gaussian</type>
-        <mean>0.0</mean>
-        <stddev>0.01</stddev>
-      </noise>
-    </ray>
-    <plugin name="lidar_controller" filename="libgazebo_ros_ray_sensor.so">
-      <topic>/scan</topic>
-      <frame_name>lidar_link</frame_name>
-    </plugin>
-  </sensor>
+<robot>
+<gazebo reference="base_link">
+<mu1>0.2</mu1>
+<mu2>0.2</mu2>
+<material>Gazebo/Black</material>
+</gazebo>
+<gazebo reference="right_wheel_back">
+<mu1>0.2</mu1>
+<mu2>0.2</mu2>
+<material>Gazebo/Yellow</material>
+</gazebo>
+<gazebo reference="right_wheel_front">
+<mu1>0.2</mu1>
+<mu2>0.2</mu2>
+<material>Gazebo/Yellow</material>
+</gazebo>
+<gazebo reference="left_wheel_back">
+<mu1>0.2</mu1>
+<mu2>0.2</mu2>
+<material>Gazebo/Yellow</material>
+</gazebo>
+<gazebo reference="left_wheel_front">
+<mu1>0.2</mu1>
+<mu2>0.2</mu2>
+<material>Gazebo/Yellow</material>
+</gazebo>
+<!--Controller for the four wheeled robot-->
+<gazebo>
+<plugin filename="ignition-gazebo-diff-drive-system" name="ignition::gazebo::systems::DiffDrive">
+    <left_joint>left_wheel_joint_front</left_joint>
+    <left_joint>left_wheel_joint_back</left_joint>
+    <right_joint>right_wheel_joint_front</right_joint>
+    <right_joint>right_wheel_joint_back</right_joint>
+    <wheel_separation>${bred+wheel_length}</wheel_separation>
+    <wheel_radius>${wheel_radius}</wheel_radius>
+    <max_linear_acceleration>0.33</max_linear_acceleration>
+    <topic>/cmd_vel</topic>
+    <frame_id>odom</frame_id>
+    <child_frame_id>base_link</child_frame_id>
+    <odom_topic>odom</odom_topic>
+    <odom_publisher_frequency>30</odom_publisher_frequency>
+    <tf_topic>tf</tf_topic>
+</plugin>
+<plugin filename="gz-sim-joint-state-publisher-system" name="gz::sim::systems::JointStatePublisher">
+    <topic>joint_states</topic>
+    <joint_name>right_wheel_joint_front</joint_name>
+    <joint_name>left_wheel_joint_front</joint_name>
+    <joint_name>right_wheel_joint_back</joint_name>
+    <joint_name>left_wheel_joint_back</joint_name>
+</plugin>
+</gazebo>
+<gazebo reference="hokuyo">
+    <sensor name="laser" type="gpu_lidar">
+        <pose>0 0 0 0 0 0</pose>
+        <always_on>true</always_on>
+        <update_rate>10</update_rate>
+        <visualize>true</visualize>
+        <topic>scan</topic>
+        <lidar>
+            <scan>
+                <horizontal>
+                <samples>360</samples>
+                <resolution>1.0</resolution>
+                <min_angle>-3.14159</min_angle>
+                <max_angle>3.14159</max_angle>
+                </horizontal>
+            </scan>
+            <range>
+                <min>0.1</min>
+                <max>10.0</max>
+                <resolution>0.01</resolution>
+            </range>
+            <noise>
+                <type>gaussian</type>
+                <mean>0.0</mean>
+                <stddev>0.01</stddev>
+            </noise>
+        </lidar>
+        <gz_frame_id>hokuyo</gz_frame_id>
+        <topic>scan</topic>
+        <plugin filename="libignition-gazebo-sensors-system.so" name="ignition::gazebo::systems::Sensors">
+            <render_engine>ogre2</render_engine>
+        </plugin>
+    </sensor>
 </gazebo>
 </robot>

Commit message: - bot with lidar added

File: bot/urdf/bot.xacro (robot description, xacro)
@@ -1,87 +1,210 @@
 <?xml version="1.0"?>
-<robot>
-<gazebo reference="base_link">
-<mu1>0.2</mu1>
-<mu2>0.2</mu2>
-<material>Gazebo/Black</material>
-</gazebo>
-<gazebo reference="right_wheel_back">
-<mu1>0.2</mu1>
-<mu2>0.2</mu2>
-<material>Gazebo/Yellow</material>
-</gazebo>
-<gazebo reference="right_wheel_front">
-<mu1>0.2</mu1>
-<mu2>0.2</mu2>
-<material>Gazebo/Yellow</material>
-</gazebo>
-<gazebo reference="left_wheel_back">
-<mu1>0.2</mu1>
-<mu2>0.2</mu2>
-<material>Gazebo/Yellow</material>
-</gazebo>
-<gazebo reference="left_wheel_front">
-<mu1>0.2</mu1>
-<mu2>0.2</mu2>
-<material>Gazebo/Yellow</material>
-</gazebo>
-<!--Controller for the four wheeled robot-->
-<gazebo>
-<plugin filename="ignition-gazebo-diff-drive-system" name="ignition::gazebo::systems::DiffDrive">
-    <left_joint>left_wheel_joint_front</left_joint>
-    <left_joint>left_wheel_joint_back</left_joint>
-    <right_joint>right_wheel_joint_front</right_joint>
-    <right_joint>right_wheel_joint_back</right_joint>
-    <wheel_separation>${bred+wheel_length}</wheel_separation>
-    <wheel_radius>${wheel_radius}</wheel_radius>
-    <max_linear_acceleration>0.33</max_linear_acceleration>
-    <topic>/cmd_vel</topic>
-    <frame_id>odom</frame_id>
-    <child_frame_id>base_link</child_frame_id>
-    <odom_topic>odom</odom_topic>
-    <odom_publisher_frequency>30</odom_publisher_frequency>
-    <tf_topic>tf</tf_topic>
-</plugin>
-<plugin filename="gz-sim-joint-state-publisher-system" name="gz::sim::systems::JointStatePublisher">
-    <topic>joint_states</topic>
-    <joint_name>right_wheel_joint_front</joint_name>
-    <joint_name>left_wheel_joint_front</joint_name>
-    <joint_name>right_wheel_joint_back</joint_name>
-    <joint_name>left_wheel_joint_back</joint_name>
-</plugin>
-</gazebo>
-<gazebo reference="hokuyo">
-    <sensor name="laser" type="gpu_lidar">
-        <pose>0 0 0 0 0 0</pose>
-        <always_on>true</always_on>
-        <update_rate>10</update_rate>
-        <visualize>true</visualize>
-        <topic>scan</topic>
-        <lidar>
-            <scan>
-                <horizontal>
-                <samples>360</samples>
-                <resolution>1.0</resolution>
-                <min_angle>-3.14159</min_angle>
-                <max_angle>3.14159</max_angle>
-                </horizontal>
-            </scan>
-            <range>
-                <min>0.1</min>
-                <max>10.0</max>
-                <resolution>0.01</resolution>
-            </range>
-            <noise>
-                <type>gaussian</type>
-                <mean>0.0</mean>
-                <stddev>0.01</stddev>
-            </noise>
-        </lidar>
-        <gz_frame_id>hokuyo</gz_frame_id>
-        <topic>scan</topic>
-        <plugin filename="libignition-gazebo-sensors-system.so" name="ignition::gazebo::systems::Sensors">
-            <render_engine>ogre2</render_engine>
-        </plugin>
-    </sensor>
-</gazebo>
+<robot xmlns:xacro="http://www.ros.org/wiki/xacro"  name="diff_drive_bot" >
+<!-- Body dimensions-->
+<xacro:property name="length" value="0.6"/>
+<xacro:property name="bred" value="0.4"/>
+<xacro:property name="height" value="0.3"/>
+<!-- Wheel dims -->
+<xacro:property name="wheel_radius" value="0.05"/>
+<xacro:property name="wheel_length" value="0.1"/>
+<xacro:property name="wheel_z" value="-0.15"/>
+<!--Material density-->
+<xacro:property name="body_density" value="2710.0"/>
+<xacro:property name="wheel_density" value="2710.0"/>
+<!--Pi constant-->
+<xacro:property name="pi_const" value="3.14159265"/>
+<!--Robot body and wheel mass-->
+<xacro:property name="body_mass" value="${body_density*length*bred*height}"/>
+<xacro:property name="wheel_mass" value="${wheel_density*pi_const*wheel_radius*wheel_radius*wheel_length}"/>
+<!-- Moment of inertia of the wheel -->
+<xacro:property name="Iz_wheel" value="${0.5*wheel_mass*wheel_radius*wheel_length}"/>
+<xacro:property name="I_wheel" value="${(1.0/12.0)*wheel_mass*(3.0*wheel_radius*wheel_radius + wheel_length*wheel_length)}"/>
+<!-- macro defining inertial section of the wheel-->
+<xacro:macro name = "inertial_wheel">
+    <inertial>
+    <origin rpy = '0 0 0' xyz= '0 0 0'/>
+    <mass value = '${wheel_mass}'/>
+    <inertia ixx = "${I_wheel}" ixy="0.0" ixz = "0.0" iyy = "${I_wheel}" iyz="0" izz="${Iz_wheel}"/>
+    </inertial>
+</xacro:macro>
+<xacro:macro name="inertial_cylinder" params="mass length radius">
+  <inertial>
+    <mass value="${mass}"/>
+    <inertia ixx="${(1/12) * mass * (3*radius*radius + length*length)}" ixy="0.0" ixz="0.0"
+                    iyy="${(1/12) * mass * (3*radius*radius + length*length)}" iyz="0.0"
+                    izz="${(1/2) * mass * (radius*radius)}" />
+  </inertial>
+</xacro:macro>
+<!--control driver with gazebo-->
+<xacro:include filename="$(find bot)/urdf/bot.gazebo"/>
+<!-- footprint link -->
+<!-- <link name="base_footprint"></link>
+<joint name="body_link_joint" type="fixed">
+  <parent link="base_footprint"/>
+  <child link="base_link"/>
+</joint> -->
+<!-- Body of the robot -->
+<link name="base_link">
+    <visual>
+        <geometry>
+          <box size="${length} ${bred} ${height}"/>
+        </geometry>
+        <material name="black">
+            <color rgba="0 0 0 1"/>
+        </material>
+    </visual>
+    <collision>
+        <geometry>
+            <box size="${length} ${bred} ${height}"/>
+        </geometry>
+        <origin rpy="0 0 0" xyz="0 0 0"/>
+    </collision>
+    <inertial>
+        <mass value = "${body_mass}"/>
+        <inertia
+            ixx = "${(1.0/12.0)*body_mass*(bred*bred + height*height)}" ixy = "0"
+            ixz = "0" iyy = "${(1.0/12.0)*body_mass*(length*length + height*height)}"
+            iyz ="0"
+            izz = "${(1.0/12.0)*body_mass*(bred*bred + length*length)}"/>
+    </inertial>
+</link>
+<!-- Joint Definition for right back wheel -->
+  <joint name="right_wheel_joint_back" type="continuous">
+    <parent link="base_link"/>
+    <child link="right_wheel_back"/>
+    <origin xyz="${-length/2+1.2*wheel_radius} ${-bred/2 - wheel_length/2} ${wheel_z}" rpy="0 0 0"/>
+    <axis xyz="0 1 0"/>
+    <limit effort="1000" velocity="1000"/>
+    <dynamics damping="1.0" friction="1.0"/>
+  </joint>
+  <!--  right back wheel -->
+  <link name="right_wheel_back">
+    <visual>
+    <origin rpy = '1.570795 0 0' xyz = '0 0 0'/>
+      <geometry>
+        <cylinder radius="${wheel_radius}" length="${wheel_length}"/> <!-- 100mm diameter wheel -->
+      </geometry>
+      <material name="grey">
+      <color rgba = '0.5 0.5 0.5 1'/>
+      </material>
+    </visual>
+    <collision>
+      <geometry>
+        <cylinder radius="${wheel_radius}" length="${wheel_length}"/>
+      </geometry>
+      <origin rpy = '1.570795 0 0' xyz = '0 0 0'/>
+    </collision>
+    <xacro:inertial_wheel/>
+  </link>
+<!-- Joint Definition for left back wheel -->
+  <joint name="left_wheel_joint_back" type="continuous">
+    <parent link="base_link"/>
+    <child link="left_wheel_back"/>
+    <origin xyz="${-length/2+1.2*wheel_radius} ${bred/2 + wheel_length/2} ${wheel_z}" rpy="0 0 0"/>
+    <axis xyz="0 1 0"/>
+    <limit effort="1000" velocity="1000"/>
+    <dynamics damping="1.0" friction="1.0"/>
+  </joint>
+  <!--  left back wheel -->
+  <link name="left_wheel_back">
+    <visual>
+    <origin rpy = '1.570795 0 0' xyz = '0 0 0'/>
+      <geometry>
+        <cylinder radius="${wheel_radius}" length="${wheel_length}"/> <!-- 100mm diameter wheel -->
+      </geometry>
+      <material name="grey">
+      <color rgba = '0.5 0.5 0.5 1'/>
+      </material>
+    </visual>
+    <collision>
+      <geometry>
+        <cylinder radius="${wheel_radius}" length="${wheel_length}"/>
+      </geometry>
+      <origin rpy = '1.570795 0 0' xyz = '0 0 0'/>
+    </collision>
+    <xacro:inertial_wheel/>
+  </link>
+<!-- Joint Definition for right front wheel -->
+  <joint name="right_wheel_joint_front" type="continuous">
+    <parent link="base_link"/>
+    <child link="right_wheel_front"/>
+    <origin xyz="${length/2-1.2*wheel_radius} ${-bred/2 - wheel_length/2} ${wheel_z}" rpy="0 0 0"/>
+    <axis xyz="0 1 0"/>
+    <limit effort="1000" velocity="1000"/>
+    <dynamics damping="1.0" friction="1.0"/>
+  </joint>
+  <!--  right front wheel -->
+  <link name="right_wheel_front">
+    <visual>
+    <origin rpy = '1.570795 0 0' xyz = '0 0 0'/>
+      <geometry>
+        <cylinder radius="${wheel_radius}" length="${wheel_length}"/> <!-- 100mm diameter wheel -->
+      </geometry>
+      <material name="grey">
+      <color rgba = '0.5 0.5 0.5 1'/>
+      </material>
+    </visual>
+    <collision>
+      <geometry>
+        <cylinder radius="${wheel_radius}" length="${wheel_length}"/>
+      </geometry>
+      <origin rpy = '1.570795 0 0' xyz = '0 0 0'/>
+    </collision>
+    <xacro:inertial_wheel/>
+  </link>
+  <!-- Joint Definition for left front wheel -->
+  <joint name="left_wheel_joint_front" type="continuous">
+    <parent link="base_link"/>
+    <child link="left_wheel_front"/>
+    <origin xyz="${length/2-1.2*wheel_radius} ${bred/2 + wheel_length/2} ${wheel_z}" rpy="0 0 0"/>
+    <axis xyz="0 1 0"/>
+    <limit effort="1000" velocity="1000"/>
+    <dynamics damping="1.0" friction="1.0"/>
+  </joint>
+  <!--  left front wheel -->
+  <link name="left_wheel_front">
+    <visual>
+    <origin rpy = '1.570795 0 0' xyz = '0 0 0'/>
+      <geometry>
+        <cylinder radius="${wheel_radius}" length="${wheel_length}"/> <!-- 100mm diameter wheel -->
+      </geometry>
+      <material name="grey">
+      <color rgba = '0.5 0.5 0.5 1'/>
+      </material>
+    </visual>
+    <collision>
+      <geometry>
+        <cylinder radius="${wheel_radius}" length="${wheel_length}"/>
+      </geometry>
+      <origin rpy = '1.570795 0 0' xyz = '0 0 0'/>
+    </collision>
+    <xacro:inertial_wheel/>
+  </link>
+  <joint name="hokuyo_joint" type="fixed">
+    <axis xyz="0 1 0" />
+    <origin xyz="0.24 0 0.175" rpy="0 0 0"/>
+    <parent link="base_link"/>
+    <child link="hokuyo"/>
+  </joint>
+  <link name="hokuyo">
+    <collision>
+      <origin xyz="0 0 0" rpy="0 0 0"/>
+      <geometry>
+    <box size="0.1 0.1 0.1"/>
+      </geometry>
+    </collision>
+    <visual>
+    <geometry>
+      <cylinder radius="0.05" length="0.05"/>
+    </geometry>
+    <material name="blue">
+      <color rgba="0 0 1 1"/>
+    </material>
+  </visual>
+    <inertial>
+      <mass value="1e-5" />
+      <origin xyz="0 0 0" rpy="0 0 0"/>
+      <inertia ixx="1e-6" ixy="0" ixz="0" iyy="1e-6" iyz="0" izz="1e-6" />
+    </inertial>
+  </link>
 </robot>
